File: KiCad_Example_Hardware/KiCad_Example_Hardware.kicad_sch (KiCad schematic)
At the start: 20 parts, among them J1 RJ45_LED_Shielded, U1 TSR_1-2450, U8 Teensy4.1_DEV-16771

Commit message: Finished 2nd H bridge
Connections:
- net FWD_PWM_2: now also U8.18 (A4); no longer U8.25 (A11)
- net FWD_PWM_4: now also U8.25 (A11); no longer U8.18 (A4)
- net RVS_PWM_2: now also U8.19 (A5); no longer U8.24 (A10)
- net RVS_PWM_4: now also U8.24 (A10); no longer U8.19 (A5)
Changed lines of the file:
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@@
     (effects (font (size 1.27 1.27)) (justify left bottom))
   )
-  (label "FWD_PWM_2" (at 111.76 161.29 180) (fields_autoplaced)
-    (effects (font (size 1.27 1.27)) (justify right bottom))
+  (label "FWD_PWM_2" (at 48.26 156.21 0) (fields_autoplaced)
+    (effects (font (size 1.27 1.27)) (justify left bottom))
   )
   (label "RVS_PWM_1" (at 116.84 83.82 0) (fields_autoplaced)
     (effects (font (size 1.27 1.27)) (justify left bottom))
   )
-  (label "FWD_PWM_4" (at 48.26 156.21 0) (fields_autoplaced)
-    (effects (font (size 1.27 1.27)) (justify left bottom))
+  (label "FWD_PWM_4" (at 111.76 161.29 180) (fields_autoplaced)
+    (effects (font (size 1.27 1.27)) (justify right bottom))
   )
   (label "RVS_PWM_1" (at 48.26 148.59 0) (fields_autoplaced)
@@
     (effects (font (size 1.27 1.27)) (justify left bottom))
   )
-  (label "RVS_PWM_4" (at 48.26 158.75 0) (fields_autoplaced)
-    (effects (font (size 1.27 1.27)) (justify left bottom))
+  (label "RVS_PWM_4" (at 111.76 163.83 180) (fields_autoplaced)
+    (effects (font (size 1.27 1.27)) (justify right bottom))
   )
   (label "FWD_PWM_3" (at 48.26 115.57 0) (fields_autoplaced)
@@
     (effects (font (size 1.27 1.27)) (justify left bottom))
   )
-  (label "RVS_PWM_2" (at 111.76 163.83 180) (fields_autoplaced)
-    (effects (font (size 1.27 1.27)) (justify right bottom))
+  (label "RVS_PWM_2" (at 48.26 158.75 0) (fields_autoplaced)
+    (effects (font (size 1.27 1.27)) (justify left bottom))
   )
   (label "FWD_PWM_2" (at 116.84 87.63 0) (fields_autoplaced)
